File: ref/flight_v2/ProPrj_AT32F435mini飞控-重制版_2026-01-28.kicad_sch (KiCad schematic)
At the start: 98 parts, among them CN1 HC-1.25-3PWT, CN2 HC-1.25-3PWT, Q1 AO6800, Q2 AO6800, SW1 MINI MSK12CO2, U1 TPS22975DSGR, U10 TPS63001DRCR, U11 PE4259-63, U12 ZX-SH1.0-4PWT, U13 ZX-MX1.25-2PWT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

Commit message: 更新prompt和完整工程
Parts:
- removed ? (x2): (no value), ProPrj_AT3-easyedapro:, symbol ProPrj_AT3-easyedapro:Short-Symbol
- removed ?: (no value), ProPrj_AT3-easyedapro:, symbol ProPrj_AT3-easyedapro:Drawing-Symbol_A4
- added ?: (no value), ProPrj_AT3-easyedapro:, symbol ProPrj_AT3-easyedapro:Drawing-Symbol_A4
- added ? (x2): (no value), ProPrj_AT3-easyedapro:, symbol ProPrj_AT3-easyedapro:Short-Symbol
Connections:
- net ELRS_RX: now also ?.2 (Pin1)
- net ELRS_TX: now also ?.2 (Pin1)
- net UART7_RX: now also ?.1 (Pin1)
- net UART7_TX: now also ?.1 (Pin1)
